File: chpndser.sch (KiCad schematic (older format))
At the start: 13 parts, among them IC101 CH340G, J101 TBLAYOUT, P101 USB_OTG, Q101 NX3008NBKW, Y101 12MHZ

Commit message: better version
Other:
- note added: ""RS232 Helper" mode is used to\naccept the inverted RX signal\nfrom the open-collector level converter."
- note added: "CH340G"
- note added: "Pandora EXT Connector and 1.8V level conversion"
- note added: "USB Connector"
- moved on the sheet: C101, C102, C103, C104, IC101, J101, P101, Q101, R101, R102, R103, R104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
