File: chpndser.kicad_pcb (KiCad board)
At the start: 2 copper layers, 12.2 x 23 mm, 13 parts, among them IC101 CH340G, J101 TBLAYOUT, P101 USB_OTG, Q101 NX3008NBKW, Y101 12MHZ

Commit message: better version
Parts:
- C103, C104: moved to B.Cu
- moved C104 15.2 mm to (147.1, 116.3), turned to 90 degrees
- moved C103 12.3 mm to (147.1, 112.7), turned to 270 degrees
- moved R104 7.90 mm to (155.4, 106.7), turned to 270 degrees
- moved R101 5.82 mm to (146.4, 108.6), turned to 270 degrees
- moved R102 3.72 mm to (147.4, 105.7), turned to 180 degrees
- moved R103 3.24 mm to (147.3, 103.4)
- moved J101 2.79 mm to (151.1, 99.1)
- moved Q101 2.57 mm to (154.4, 103.4)
- moved Y101 2.17 mm to (151.4, 111.3), turned to 270 degrees
- moved C102 1.66 mm to (148.1, 108.6), turned to 270 degrees
Routing:
- net /CHTX: track 5.36 -> 18.2 mm
- net /CHRX: track 13.7 -> 5.37 mm, vias 2 -> 1
- net +5V: track 23.9 -> 16.4 mm
- net GND: track 59.7 -> 53.5 mm, vias 5 -> 4
- net Net-(C104-Pad1): track 13.2 -> 18.8 mm
- net Net-(J101-Pad4): track 9.36 -> 7.90 mm
- net /DP: track 9.02 -> 10.4 mm
- net Net-(C102-Pad1): track 5.24 -> 6.10 mm
- net /DM: track 9.11 -> 9.63 mm
Other:
- board size 12.2 x 23 mm -> 11.7 x 20.2 mm
- board text added: "160315"
- board text added: "PND DBG USB"

Commit message: First public release version
Routing:
- net +5V: track 16.4 -> 17.4 mm
- net Net-(J101-Pad4): track 7.90 -> 7.27 mm
Other:
- outline, holes or cut-outs redrawn
- board text added: "160421"
- board text removed: "160315"
